File: RP2350B-Flight-controller.kicad_pcb (KiCad board)
At the start: 2 copper layers, 30.2 x 39.8 mm, 136 parts, among them Q1 FS3400, Q2 FS3400, Q3 FS3400, Q4 FS3400, SW1 KMR221GLFS, SW2 KMR221GLFS, U1 USBLC6-2SC6, U2 INA180A2, X1 Conn_Coaxial, X2 USB_C_Receptacle_USB2.0_14P, Y1 16MHz, Y2 16MHz

Commit message: rev0 ready
Parts:
- added G***: LOGO, LOGO, F.Cu at (80.5, 38.7)
- added G***: LOGO, LOGO, F.Cu at (89.2, 62.8)
- added G***: LOGO, LOGO, F.Cu at (80.6, 36.1)
- added G***: LOGO, LOGO, F.Cu at (79.8, 47.6)
- added G***: LOGO, LOGO, B.Cu at (83.1, 48.3)
- added TP1: TestPoint, TestPoint:TestPoint_Pad_D1.0mm, F.Cu at (92.4, 63.5)
- added TP2: TestPoint, TestPoint:TestPoint_Pad_D1.0mm, F.Cu at (92.4, 62.1)
- added TP3: TestPoint, TestPoint:TestPoint_Pad_D1.0mm, F.Cu at (93.8, 63.5)
- added TP4: TestPoint, TestPoint:TestPoint_Pad_D1.0mm, F.Cu at (93.8, 62.1)
- added TP5: TestPoint, TestPoint:TestPoint_Pad_D1.0mm, F.Cu at (95.2, 63.5)
- added TP6: TestPoint, TestPoint:TestPoint_Pad_D1.0mm, F.Cu at (95.2, 62.1)
- added TP7: TestPoint, TestPoint:TestPoint_Pad_D1.0mm, F.Cu at (96.8, 63.5)
- added TP8: TestPoint, TestPoint:TestPoint_Pad_D1.0mm, F.Cu at (96.8, 62.1)
- R14: value 10K -> 1K
- moved C28 14.7 mm to (85.1, 47.8), turned to 90 degrees
- moved C25 13.7 mm to (92.5, 54.4), turned to 0 degrees
- moved C26 7.16 mm to (79.4, 54.7)
- moved R21 1.30 mm to (77.6, 61.9)
- moved C41 0.30 mm to (88.7, 47.8)
- renumbered TP2 to TP10, TP3 to TP11, TP4 to TP12, TP5 to TP13, TP6 to TP14, TP7 to TP15, TP8 to TP16, TP9 to TP17, TP10 to TP18, TP11 to TP19, TP12 to TP20, TP13 to TP21, TP14 to TP22, TP15 to TP23, TP16 to TP24, TP17 to TP25, TP18 to TP26, TP1 to TP9
Connections:
- DD4 pad 1: unconnected-(DD4-GPIO4-Pad1) -> Net-(DD4-GPIO4)
- DD4 pad 17: unconnected-(DD4-GPIO17-Pad17) -> LED1
- DD4 pad 18: unconnected-(DD4-GPIO18-Pad18) -> LED2
- DD4 pad 2: unconnected-(DD4-GPIO5-Pad2) -> Net-(DD4-GPIO5)
- DD4 pad 3: unconnected-(DD4-GPIO6-Pad3) -> Net-(DD4-GPIO6)
- DD4 pad 4: unconnected-(DD4-GPIO7-Pad4) -> Net-(DD4-GPIO7)
- DD4 pad 43: LED1 -> unconnected-(DD4-GPIO34-Pad43)
- DD4 pad 44: LED2 -> unconnected-(DD4-GPIO35-Pad44)
- DD4 pad 6: unconnected-(DD4-GPIO8-Pad6) -> Net-(DD4-GPIO8)
- DD4 pad 7: unconnected-(DD4-GPIO9-Pad7) -> Net-(DD4-GPIO9)
- DD4 pad 8: unconnected-(DD4-GPIO10-Pad8) -> Net-(DD4-GPIO10)
- DD4 pad 80: unconnected-(DD4-GPIO3-Pad80) -> Net-(DD4-GPIO3)
Routing:
- net 3.3V: track 0.00 -> 108.5 mm, vias 0 -> 22
- net RUN: track 0.00 -> 30.7 mm, vias 0 -> 2
- net V_Motors: track 0.00 -> 27.9 mm, vias 0 -> 38
- net Net-(DD4-SWCLK): track 0.00 -> 17.6 mm, vias 0 -> 2
- net Net-(DD4-SWDIO): track 0.00 -> 16.8 mm, vias 0 -> 2
- net Motor_voltage: track 0.00 -> 16.7 mm, vias 0 -> 2
- net Motor_1: track 0.00 -> 16.6 mm
- net LED1: track 0.00 -> 15.4 mm
- net LED2: track 0.00 -> 13.8 mm
- net Net-(DD4-GPIO9): track 0.00 -> 12.0 mm
- net Motor_2: track 0.00 -> 11.9 mm
- net Net-(DD4-GPIO10): track 0.00 -> 11.1 mm
- net Net-(DD4-GPIO11): track 0.00 -> 9.91 mm
- net NRF_CE: track 4.13 -> 13.7 mm, vias 0 -> 2
- net Net-(DD4-GPIO8): track 0.00 -> 9.45 mm
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- added copper zone on B.Cu, net 3.3V
- added copper zone on F.Cu, net 3.3V
- added copper zone on B.Cu, net Earth
- added copper zone on F.Cu, net Earth
- added copper zone on F.Cu, net Net-(DD4-ADC_AVDD)
- added copper zone on F.Cu, net Net-(DD4-DVDD_1)
- added copper zone on F.Cu, net Net-(DD4-VREG_LX)
- added copper zone on B.Cu, net VCC-5V
- added copper zone on F.Cu, net VCC-5V
- added copper zone on B.Cu, net V_Motors
- added copper zone on F.Cu, net V_Motors
Other:
- board text added: "1"
- board text added: "2"
- board text added: "3"
- board text added: "4"
- board text added: "@madjogger"
- board text added: "RP2350B Flight"
- board text added: "boot"
- board text added: "controller"
- board text added: "rst"

Commit message: connected 21 pin of nrf24l01+ to GND
Connections:
- DD1 pad 21: (no net) -> Earth
Changed lines of the file:
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@@
 			(property pad_prop_heatsink)
 			(layers "F.Cu" "F.Mask")
+			(net 2 "Earth")
+			(pinfunction "PAD")
+			(pintype "power_in")
 			(zone_connect 2)
 		)
@@
 		(polygon
 			(pts
-				(xy 83.3 59.5) (xy 82.9 59.9) (xy 82.6 59.9) (xy 82.4 60.1) (xy 82.4 60.8) (xy 82 61.2) (xy 82 61.2)
-				(xy 82 61.75) (xy 82.1 61.9) (xy 82.7 61.9) (xy 82.72 61.7) (xy 82.72 61.48) (xy 82.9 61.3) (xy 83.2 61.3)
-				(xy 83.3 61.2) (xy 83.3 60.3) (xy 83.8 59.8) (xy 83.8 59) (xy 83.7 58.9) (xy 83.4 58.9) (xy 83.3 59)
+				(xy 83.3 59.5) (xy 82.9 59.9) (xy 82.6 59.9) (xy 82.4 60.1) (xy 82.4 60.8) (xy 82 61.2) (xy 82 61.75)
+				(xy 82.1 61.9) (xy 82.7 61.9) (xy 82.72 61.7) (xy 82.72 61.48) (xy 82.9 61.3) (xy 83.2 61.3) (xy 83.3 61.2)
+				(xy 83.3 60.3) (xy 83.8 59.8) (xy 83.8 59) (xy 83.7 58.9) (xy 83.4 58.9) (xy 83.3 59)
 			)
 		)
