File: RP2350B-Flight-controller.kicad_sch (KiCad schematic)
At the start: 7 parts, among them Q1 FS3400, U1 INA180A2

Commit message: schematics and component placement done
Parts:
- removed DD2: CC2590RGVTG4, CC2590RG:CC2590RG, symbol CC2590RGVTG4:CC2590RGVTG4
- added C1, C2, C32, C39: 22pF, Capacitor_SMD:C_0201_0603Metric, symbol Device:C
- added C10, C16, C19, C21, C23: 1.5pF, Capacitor_SMD:C_0201_0603Metric, symbol Device:C
- added C11: 4.7pF, Capacitor_SMD:C_0201_0603Metric, symbol Device:C
- added C12: 1nF, Capacitor_SMD:C_0201_0603Metric, symbol Device:C
- added C13: 1pF, Capacitor_SMD:C_0201_0603Metric, symbol Device:C
- added C14: 0.3pF, Capacitor_SMD:C_0201_0603Metric, symbol Device:C
- added C15, C18, C22, C24, C25, C26, C27, C29, C35, C36, C37, C38, C40, C41, C42, C43, C45, C46, C48, C49, C5, C50, C6, C7: 4.7uF, Capacitor_SMD:C_0201_0603Metric, symbol Device:C
- added C17: 220pF, Capacitor_SMD:C_0201_0603Metric, symbol Device:C
- added C20, C30, C31, C33, C34, C4, C44: 100nF, Capacitor_SMD:C_0201_0603Metric, symbol Device:C
- added C28, C9: 10nF, Capacitor_SMD:C_0201_0603Metric, symbol Device:C
- added C3: 33nF, Capacitor_SMD:C_0201_0603Metric, symbol Device:C
- added C47, C51, C52, C53, C54: 22uF, Capacitor_SMD:C_0402_1005Metric, symbol Device:C
- added C8: 2.2nF, Capacitor_SMD:C_0201_0603Metric, symbol Device:C
- added D1, D2, D3: LED 0402, LED_SMD:LED_0402_1005Metric, symbol Device:LED
- added D4: SS54F, PCM_Diode_SMD_AKL:D_SMAFL, symbol PCM_Diode_Schottky_AKL:SS54F
- added D5, D6, D7, D8: B5819W, Diode_SMD:D_SOD-123, symbol PCM_Diode_Schottky_AKL:D_Schottky_Generic
- added DA1: RFX2401C, RFX2401C:RFX2401C, symbol RFX2401C:RFX2401C
- added DD3: W25Q16JVUXIQ_TR, W25Q16JVUXIQ:W25Q16JVUXIQ, symbol W25Q16JVUXIQ_TR:W25Q16JVUXIQ_TR
- added DD5: BCT2057ELT33, BCT2057ELTAJ:BCT2057ELTAJ, symbol BCT2057ELTAJ:BCT2057ELTAJ-TR
- added L1: 8.2nH, Inductor_SMD:L_0201_0603Metric, symbol Device:L
- added L2: 3.9nH, Inductor_SMD:L_0201_0603Metric, symbol Device:L
- added L3: 2.7nH, Inductor_SMD:L_0201_0603Metric, symbol Device:L
- added L4, L5: 2.4nH, Inductor_SMD:L_0201_0603Metric, symbol Device:L
- added L6: VHF160808H33NJT, Inductor_SMD:L_0603_1608Metric, symbol Device:L
- added L7: FHW0603UF3R3JST, Inductor_SMD:L_0603_1608Metric, symbol Device:L
- added Q2, Q3, Q4: FS3400, Package_TO_SOT_SMD:SOT-23, symbol Device:Q_NMOS
- added R1, R15: 1M, PCM_Resistor_SMD_AKL:R_0201_0603Metric, symbol Device:R
- added R10: 20K, PCM_Resistor_SMD_AKL:R_0201_0603Metric, symbol Device:R
- added R11, R13, R2, R3, R4, R6, R7, R8, R9: 1K, PCM_Resistor_SMD_AKL:R_0201_0603Metric, symbol Device:R
- added R12, R14, R18, R19, R27, R28, R29, R30: 10K, PCM_Resistor_SMD_AKL:R_0201_0603Metric, symbol Device:R
- added R16, R17: 27R, PCM_Resistor_SMD_AKL:R_0201_0603Metric, symbol Device:R
- added R21, R22: 5.1K, PCM_Resistor_SMD_AKL:R_0201_0603Metric, symbol Device:R
- added R23, R24, R25, R26: 220R, PCM_Resistor_SMD_AKL:R_0201_0603Metric, symbol Device:R
- added R31: 0R, PCM_Resistor_SMD_AKL:R_0805_2012Metric, symbol Device:R
- added R5: 22K, PCM_Resistor_SMD_AKL:R_0201_0603Metric, symbol Device:R
- added SW1, SW2: KMR221GLFS, Button_Switch_SMD:SW_SPST_PTS810, symbol Switch:SW_Push
- added TP1, TP2, TP3, TP4, TP5, TP6, TP7, TP8: TestPoint, TestPoint:TestPoint_Pad_D1.0mm, symbol Connector:TestPoint
- added TP10, TP11, TP12, TP13, TP14, TP15, TP16, TP17, TP18, TP9: TestPoint, TestPoint:TestPoint_Pad_D1.5mm, symbol Connector:TestPoint
- added U1: USBLC6-2SC6, Package_TO_SOT_SMD:SOT-23-6, symbol Power_Protection:USBLC6-2SC6
- added X1: Conn_Coaxial, Connector_Coaxial:U.FL_Molex_MCRF_73412-0110_Vertical, symbol Connector:Conn_Coaxial
- added X2: USB_C_Receptacle_USB2.0_14P, Connector_USB:USB_C_Receptacle_GCT_USB4105-xx-A_16P_TopMnt_Horizontal, symbol Connector:USB_C_Receptacle_USB2.0_14P
- added Y1, Y2: 16MHz, Crystal:Crystal_SMD_3225-4Pin_3.2x2.5mm, symbol Device:Crystal_GND24
- renumbered DD to DD1, DD1 to DD2, DD1 to DD4, R1 to R20, U1 to U2
Connections:
- net Motor_current: now reaches U2.1
- net Motor_current: now also DD4.49 (GPIO40_ADC0)
- net Earth: now reaches U2.2 (GND)
- net Earth: now also DD1.14 (VSS), DD1.17 (VSS), DD1.20 (VSS), DD1.8 (VSS), DD2.6 (GND), DD2.7 (GND), DD4.62 (VREG_PGND), DD4.81 (GND), Q1.2 (S), C1.2, C11.2, C12.2, C13.2, C14.2, C15.2, C16.2, C17.2, C18.2, C19.2, C2.2, C20.2, C21.2, C22.2, C23.2, C24.2, C25.2, C26.2, C27.1, C28.2, C29.1, C3.2, C30.2, C31.2, C32.2, C33.2, C34.2, C35.2, C36.2, C37.2, C38.2, C39.2, C4.2, C40.2, C41.2, C42.2, C43.2, C44.2, C45.2, C46.2, C47.2, C48.2, C49.2, C5.2, C50.2, C51.2, C52.2, C53.2, C54.2, C6.2, C7.2, C8.2, C9.2, D1.1 (K), D2.1 (K), D3.1 (K), D4.2 (A), DA1.11 (GND_5), DA1.17 (GND_6), DA1.2 (GND_1), DA1.3 (GND_2), DA1.8 (GND_3), DA1.9 (GND_4), DD3.4 (GND), DD5.0 (EP), DD5.3 (GND), Q2.2 (S), Q3.2 (S), Q4.2 (S), R10.2, R19.1, R2.1, R21.1, R22.1, R27.1, R28.1, R29.1, R3.1, R30.1, R4.1, R5.1, SW1.1, SW2.1, TP18.1, U1.2 (GND), X1.2 (Ext), X2.A1 (GND), X2.A12 (GND), X2.B1 (GND), X2.B12 (GND), X2.S1 (SHIELD), Y1.2, Y1.4, Y2.2, Y2.4
- net VCC-5V: now reaches U2.3 (+)
- net VCC-5V: now also R20.1, C42.1, C43.1, C44.1, C45.1, C46.1, D4.1 (K), DD5.4 (EN), DD5.6 (IN), R31.1, U1.5 (VBUS), X2.A4 (VBUS), X2.A9 (VBUS), X2.B4 (VBUS), X2.B9 (VBUS)
- net V_Motors: now reaches U2.4 (-)
- net V_Motors: now also R20.2, C51.1, C52.1, C53.1, C54.1, D5.1 (K), D6.1 (K), D7.1 (K), D8.1 (K), R18.2, TP11.1, TP13.1, TP15.1, TP9.1
- net 3.3V: now reaches U2.5 (V+)
- net 3.3V: now also DD1.15 (VDD), DD1.18 (VDD), DD1.7 (VDD), DD2.5 (VDDIO), DD2.8 (VDD), DD4.15 (IOVDD_2), DD4.24 (IOVDD_3), DD4.29 (IOVDD_4), DD4.41 (IOVDD_5), DD4.5 (IOVDD_1), DD4.50 (IOVDD_6), DD4.60 (IOVDD_7), DD4.64 (VREG_VIN), DD4.68 (USB_OTP_VDD), DD4.69 (QSPI_IOVDD), DD4.76 (IOVDD_8), C12.1, C15.1, C17.1, C18.1, C20.1, C22.1, C30.1, C31.1, C33.1, C34.1, C35.1, C36.1, C37.1, C38.1, C4.1, C40.1, C41.1, C47.1, C48.1, C49.1, C5.1, C50.1, C6.1, C7.1, C9.1, DA1.16 (VDD_2), DD3.8 (VCC), DD5.1 (OUT), L6.1, R11.1, R12.2
- net NRF_CE: now reaches DD1.1 (CE)
- net NRF_CE: now also DD4.39 (GPIO31), R9.1
- net at DD1.10 (XC1): now also C2.1, R1.2, Y1.3
- net VDD_PA: now reaches DD1.11 (VDD_PA)
- net VDD_PA: now also C11.1, C8.1, L3.2, R8.1
- net at DD1.12 (ANT1): now also L1.2, L3.1
- net at DD1.13 (ANT2): now also L1.1, L2.1
- net at DD1.16 (IREF): now also R5.2
- net at DD1.19 (DVDD): now also C3.1
- net NRF_CS: now reaches DD1.2 (CSN)
- net NRF_CS: now also DD4.38 (GPIO30)
- net SPI_SCK: now reaches DD1.3 (SCK)
- net SPI_SCK: now also DD4.37 (GPIO29)
- net SPI_MOSI: now reaches DD1.4 (MOSI)
- net SPI_MOSI: now also DD4.28 (GPIO27)
- net SPI_MISO: now reaches DD1.5 (MISO)
- net SPI_MISO: now also DD4.36 (GPIO28)
- net NRF_IRQ: now reaches DD1.6 (IRQ)
- net NRF_IRQ: now also DD4.40 (GPIO32)
- net at DD1.9 (XC2): now also C1.1, R1.1, Y1.1
- net at DD4.10 (DVDD_1): now also DD4.32 (DVDD_2), DD4.51 (DVDD_3), DD4.65 (VREG_FB), C24.1, C25.1, C26.1, C28.1, L7.2
- net at DD4.11 (GPIO12): now also TP2.1
- net at DD4.12 (GPIO13): now also TP3.1
- net at DD4.13 (GPIO14): now also TP4.1
- net at DD4.14 (GPIO15): now also TP5.1
- net at DD4.16 (GPIO16): now also TP6.1
- net SPI2_MISO: now reaches DD4.19 (GPIO19)
- net SPI2_MISO: now also DD2.1 (SDO/SA0)
- net IMU_INT1: now reaches DD4.20 (GPIO20)
- net IMU_INT1: now also DD2.4 (INT1)
- net IMU_INT2: now reaches DD4.21 (GPIO21)
- net IMU_INT2: now also DD2.9 (INT2)
- net SPI2_MOSI: now reaches DD4.22 (GPIO22)
- net SPI2_MOSI: now also DD2.14 (SDA)
- net SPI2_SCK: now reaches DD4.23 (GPIO23)
- net SPI2_SCK: now also DD2.13 (SCL)
- net at DD4.30 (XIN): now also C39.1, R15.1, Y2.1
- net at DD4.31 (XOUT): now also C32.1, R15.2, Y2.3
- net at DD4.33 (SWCLK): now also TP8.1
- net at DD4.34 (SWDIO): now also TP7.1
- net RUN: now reaches DD4.35 (RUN)
- net RUN: now also R12.1, R13.1
- net LED1: now reaches DD4.43 (GPIO34)
- net LED1: now also R7.1
- net LED2: now reaches DD4.44 (GPIO35)
- net LED2: now also R6.1
- net Motor_1: now reaches DD4.45 (GPIO36)
- net Motor_1: now also R23.1
- net Motor_2: now reaches DD4.46 (GPIO37)
- net Motor_2: now also R24.1
- net Motor_3: now reaches DD4.47 (GPIO38)
- net Motor_3: now also R25.1
- net Motor_4: now reaches DD4.48 (GPIO39)
- net Motor_4: now also R26.1
- net Motor_voltage: now reaches DD4.52 (GPIO41_ADC1)
- net Motor_voltage: now also R18.1, R19.2
- net at DD4.59 (ADC_AVDD): now also DD4.61 (VREG_AVDD), C27.2, C29.2, L6.2
- net at DD4.63 (VREG_LX): now also L7.1
- net USB_R-: now reaches DD4.66 (USB_DM)
- net USB_R-: now also R17.1
- net USB_R+: now reaches DD4.67 (USB_DP)
- net USB_R+: now also R16.1
- net QSPI_SD3: now reaches DD4.70 (QSPI_SD3)
- net QSPI_SD3: now also DD3.7 (IO3)
- net QSPI_SCLK: now reaches DD4.71 (QSPI_SCLK)
- net QSPI_SCLK: now also DD3.6 (CLK)
- net QSPI_SD0: now reaches DD4.72 (QSPI_SD0)
- net QSPI_SD0: now also DD3.5 (DI(IO0))
- net QSPI_SD2: now reaches DD4.73 (QSPI_SD2)
- net QSPI_SD2: now also DD3.3 (IO2)
- net QSPI_SD1: now reaches DD4.74 (QSPI_SD1)
- net QSPI_SD1: now also DD3.2 (DO(IO1))
- net QSPI_SS: now reaches DD4.75 (QSPI_SS)
- net QSPI_SS: now also DD3.1 (~{CS}), R14.1
- net at DD4.9 (GPIO11): now also TP1.1
- net at DD2.12 (CS): now also R4.2
- net at DD2.2 (SDX): now also R2.2
- net at DD2.3 (SCX): now also R3.2
- new net: C19.1, C21.1, L4.2, L5.1
- new net: R13.2, SW1.2
- new net: Q4.1 (G), R26.2, R30.2
- new net: D6.2 (A), Q2.3 (D), TP12.1
- new net: R22.2, X2.B5 (CC2)
- new net: C14.1, C16.1, DA1.10 (ANT), L4.1
- new net: D3.2 (A), R11.2
- new net: R14.2, SW2.2
- new net: Q3.1 (G), R25.2, R29.2
- new net: D7.2 (A), Q3.3 (D), TP14.1
- new net: Q2.1 (G), R24.2, R28.2
- new net: Q1.1 (G), R23.2, R27.2
- new net: C23.1, L5.2, X1.1 (In)
- new net: D8.2 (A), Q4.3 (D), TP16.1
- new net: C10.1, L2.2
- new net: C10.2, C13.1, DA1.4 (TXRX)
- new net: D5.2 (A), Q1.3 (D), TP10.1
- new net: D1.2 (A), R6.2
- new net: D2.2 (A), R7.2
- new net: DA1.6 (RXEN), R10.1, R9.2
- new net: DA1.5 (TXEN), R8.2
- new net: R21.2, X2.A5 (CC1)
- new net USB_Conn+: U1.6 (I/O1), X2.A6 (D+), X2.B6 (D+)
- new net USB_Conn-: U1.4 (I/O2), X2.A7 (D-), X2.B7 (D-)
- new net USB_ESD+: R16.2, U1.1 (I/O1)
- new net USB_ESD-: R17.2, U1.3 (I/O2)
- new net VBAT: R31.2, TP17.1
- no-connect marks 0 -> 25
Other:
- moved on the sheet: DD1, DD2, DD4, R20

Commit message: rev0 ready
Parts:
- added TP1, TP2, TP3, TP4, TP5, TP6, TP7, TP8: TestPoint, TestPoint:TestPoint_Pad_D1.0mm, symbol Connector:TestPoint
- R14: value 10K -> 1K
- renumbered TP2 to TP10, TP3 to TP11, TP4 to TP12, TP5 to TP13, TP6 to TP14, TP7 to TP15, TP8 to TP16, TP9 to TP17, TP10 to TP18, TP11 to TP19, TP12 to TP20, TP13 to TP21, TP14 to TP22, TP15 to TP23, TP16 to TP24, TP17 to TP25, TP18 to TP26, TP1 to TP9
Connections:
- net LED1: now also DD4.17 (GPIO17); no longer DD4.43 (GPIO34)
- net LED2: now also DD4.18 (GPIO18); no longer DD4.44 (GPIO35)
- net at DD4.1 (GPIO4): now also TP2.1
- net at DD4.2 (GPIO5): now also TP3.1
- net at DD4.3 (GPIO6): now also TP4.1
- net at DD4.4 (GPIO7): now also TP5.1
- net at DD4.6 (GPIO8): now also TP6.1
- net at DD4.7 (GPIO9): now also TP7.1
- net at DD4.8 (GPIO10): now also TP8.1
- net at DD4.80 (GPIO3): now also TP1.1
- no-connect marks 25 -> 17

Commit message: connected 21 pin of nrf24l01+ to GND
Connections:
- net Earth: now also DD1.21 (PAD)
Changed lines of the file:
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@@
 		(pin "16"
+		)
+		(pin "21"
 		)
 		(instances
